Commit message: updte init config

File: panda_resources/panda_moveit_config/config/panda.urdf.xacro (robot description, xacro)
@@ -9,4 +9,4 @@
     <xacro:include filename="panda_hand.ros2_control.xacro" />
     <xacro:panda_ros2_control name="PandaFakeSystem" initial_positions_file="$(arg initial_positions_file)" ros2_control_hardware_type="$(arg ros2_control_hardware_type)"/>
-    <xacro:panda_hand_ros2_control name="PandaHandFakeSystem" ros2_control_hardware_type="$(arg ros2_control_hardware_type)"/>
+    <xacro:panda_hand_ros2_control name="PandaHandFakeSystem" initial_positions_file="$(arg initial_positions_file)" ros2_control_hardware_type="$(arg ros2_control_hardware_type)"/>
 </robot>

File: panda_resources/panda_moveit_config/config/panda_hand.ros2_control.xacro (robot description, xacro)
@@ -1,5 +1,6 @@
 <?xml version="1.0"?>
 <robot xmlns:xacro="http://www.ros.org/wiki/xacro">
-    <xacro:macro name="panda_hand_ros2_control" params="name ros2_control_hardware_type">
+    <xacro:macro name="panda_hand_ros2_control" params="name initial_positions_file ros2_control_hardware_type">
+        <xacro:property name="initial_positions" value="${xacro.load_yaml(initial_positions_file)['initial_positions']}"/>
         <ros2_control name="${name}" type="system">
             <hardware>
@@ -28,5 +29,5 @@
                 </xacro:unless>
                 <state_interface name="position">
-                  <param name="initial_value">0.0</param>
+                  <param name="initial_value">${initial_positions['panda_finger_joint1']}</param>
                 </state_interface>
                 <state_interface name="velocity">
@@ -48,5 +49,5 @@
                 </xacro:unless>
                 <state_interface name="position">
-                  <param name="initial_value">0.0</param>
+                  <param name="initial_value">${initial_positions['panda_finger_joint2']}</param>
                 </state_interface>
                 <state_interface name="velocity">

Commit message: update code

File: panda_resources/panda_moveit_config/config/panda.urdf.xacro (robot description, xacro)
@@ -5,4 +5,12 @@
     <!-- Import panda urdf file -->
     <xacro:include filename="$(find moveit_resources_panda_description)/urdf/panda.urdf" />
+    <!-- Define an explicit FT frame attached to panda_hand. -->
+    <link name="sensor_fts"/>
+    <joint name="sensor_fts_joint" type="fixed">
+        <parent link="panda_hand"/>
+        <!-- Co-located with panda_hand; tweak xyz/rpy if you want an offset. -->
+        <origin xyz="0 0 0" rpy="0 0 0"/>
+        <child link="sensor_fts"/>
+    </joint>
     <!-- Import panda ros2_control description -->
     <xacro:include filename="panda.ros2_control.xacro" />
